Commit message: adapted to new requirement of hw interface in joint tag

File: mico_description/urdf/arms/mico_arm.urdf.xacro (robot description, xacro)
@@ -117,5 +117,7 @@
     <transmission name="j1_trans">
 	 <type>transmission_interface/SimpleTransmission</type>
-     <joint name="mico_joint_1" />
+     <joint name="mico_joint_1">
+        <hardwareInterface>EffortJointInterface</hardwareInterface>
+     </joint>
      <actuator name="j1_motor">
 	    <hardwareInterface>EffortJointInterface</hardwareInterface>
@@ -168,5 +170,7 @@
     <transmission name="j2_trans">
 	 <type>transmission_interface/SimpleTransmission</type>
-     <joint name="mico_joint_2" />
+     <joint name="mico_joint_2">
+        <hardwareInterface>EffortJointInterface</hardwareInterface>
+     </joint>
      <actuator name="j2_motor">
 	    <hardwareInterface>EffortJointInterface</hardwareInterface>
@@ -219,5 +223,7 @@
     <transmission name="j3_trans">
 	 <type>transmission_interface/SimpleTransmission</type>
-     <joint name="mico_joint_3" />
+     <joint name="mico_joint_3">
+        <hardwareInterface>EffortJointInterface</hardwareInterface>
+     </joint>
      <actuator name="j3_motor">
 	    <hardwareInterface>EffortJointInterface</hardwareInterface>
@@ -270,5 +276,7 @@
     <transmission name="j4_trans">
 	 <type>transmission_interface/SimpleTransmission</type>
-     <joint name="mico_joint_4" />
+     <joint name="mico_joint_4">
+        <hardwareInterface>EffortJointInterface</hardwareInterface>
+     </joint>
      <actuator name="j4_motor">
 	    <hardwareInterface>EffortJointInterface</hardwareInterface>
@@ -321,5 +329,7 @@
     <transmission name="j5_trans">
 	 <type>transmission_interface/SimpleTransmission</type>
-     <joint name="mico_joint_5" />
+     <joint name="mico_joint_5">
+        <hardwareInterface>EffortJointInterface</hardwareInterface>
+     </joint>
      <actuator name="j5_motor">
 	    <hardwareInterface>EffortJointInterface</hardwareInterface>
@@ -372,5 +382,7 @@
     <transmission name="j6_trans">
 	 <type>transmission_interface/SimpleTransmission</type>
-     <joint name="mico_joint_6" />
+     <joint name="mico_joint_6">
+        <hardwareInterface>EffortJointInterface</hardwareInterface>
+     </joint>
      <actuator name="j6_motor">
 	    <hardwareInterface>EffortJointInterface</hardwareInterface>
@@ -423,5 +435,7 @@
     <transmission name="jf1_trans">
 	 <type>transmission_interface/SimpleTransmission</type>
-     <joint name="mico_joint_finger_1" />
+     <joint name="mico_joint_finger_1">
+        <hardwareInterface>EffortJointInterface</hardwareInterface>
+     </joint>
      <actuator name="jf1_motor">
 	    <hardwareInterface>EffortJointInterface</hardwareInterface>
@@ -474,5 +488,7 @@
     <transmission name="jf2_trans">
 	 <type>transmission_interface/SimpleTransmission</type>
-     <joint name="mico_joint_finger_2" />
+     <joint name="mico_joint_finger_2">
+        <hardwareInterface>EffortJointInterface</hardwareInterface>
+     </joint>
      <actuator name="jf2_motor">
 	    <hardwareInterface>EffortJointInterface</hardwareInterface>

Commit message: modifications to the moveit_config to use the follow_joint_trajectory controller

File: mico_description/urdf/arms/mico_arm.urdf.xacro (robot description, xacro)
@@ -8,9 +8,9 @@
 	<xacro:property name="j3_motor_torque_constant" value="50.0"/>
 	<xacro:property name="j4_mechanical_reduction" value="1.0"/>
-	<xacro:property name="j4_motor_torque_constant" value="5.0"/>
+	<xacro:property name="j4_motor_torque_constant" value="15.0"/>
 	<xacro:property name="j5_mechanical_reduction" value="1.0"/>
-	<xacro:property name="j5_motor_torque_constant" value="5.0"/>
+	<xacro:property name="j5_motor_torque_constant" value="15.0"/>
 	<xacro:property name="j6_mechanical_reduction" value="1.0"/>
-	<xacro:property name="j6_motor_torque_constant" value="5.0"/>
+	<xacro:property name="j6_motor_torque_constant" value="15.0"/>
 	<xacro:property name="jf1_mechanical_reduction" value="1.0"/>
 	<xacro:property name="jf1_motor_torque_constant" value="5.0"/>
@@ -35,6 +35,6 @@
 	<xacro:property name="joint_effort_limit" value="60.0"/>
 	<xacro:property name="joint_velocity_limit" value="2.9217"/>
-	<xacro:property name="joint_damping" value="0.7"/>
-	<xacro:property name="joint_friction" value="0.5"/>
+        <xacro:property name="joint_damping" value="0.7"/>
+        <xacro:property name="joint_friction" value="0.5"/>
   <!--
   <property name="link_end_effector"   value="mico_end_effector" />
@@ -46,7 +46,7 @@
 	<link name="mico_link_base">
 		<inertial>
-		  <mass value="0.506" />
-		  <origin xyz="-0.05161 0 -0.003" />
-		  <inertia  ixx="0.0014526484" ixy="0.0"  ixz="-8.792613e-005" iyy="0.0018217854" iyx="0.0"  iyz="0.0" izz="0.0008987159" />
+		  <mass value="1" />
+		  <origin xyz="0.0 0.0 0.0" />
+		  <inertia  ixx="0.1" ixy="0.0"  ixz="0.0" iyy="0.1" iyx="0.0"  iyz="0.0" izz="0.1" />
 		</inertial>
 		<visual>
@@ -76,7 +76,7 @@
     <link name="mico_link_1">
 		<inertial>
-		  <mass value="0.7" />
+		  <mass value="1" />
 		  <origin xyz="0.07155 0.00229 -0.00028" />
-		  <inertia  ixx="0.0018430902" ixy="0.0001075379"  ixz="2.683183e-005"  iyy="0.0023530852"  iyz="4.5192e-007"  izz="0.0016327528" />
+		  <inertia  ixx="0.1" ixy="0.0"  ixz="0.0"  iyy="0.1"  iyz="0.0"  izz="0.1" />
 		</inertial>
 		<visual>
@@ -121,7 +121,6 @@
      </joint>
      <actuator name="j1_motor">
-	    <hardwareInterface>EffortJointInterface</hardwareInterface>
-        <mechanicalReduction>${j1_mechanical_reduction}</mechanicalReduction>
-		<motorTorqueConstant>${j1_motor_torque_constant}</motorTorqueConstant>
+            <mechanicalReduction>${j1_mechanical_reduction}</mechanicalReduction>
+	    <motorTorqueConstant>${j1_motor_torque_constant}</motorTorqueConstant>
 	 </actuator>
     </transmission>
@@ -129,7 +128,7 @@
 	<link name="mico_link_2">
 		<inertial>
-		  <mass value="0.429" />
+		  <mass value="1" />
 		  <origin xyz="0.06076 0 -0.00014" />
-		  <inertia  ixx="0.0011551458" ixy="-6.3e-010"  ixz="2.519546e-005"  iyy="0.0015754353"  iyz="-7.6e-010"  izz="0.0007798411" />
+		  <inertia  ixx="0.1" ixy="0.0"  ixz="0.0"  iyy="0.1"  iyz="0.0"  izz="0.1" />
 		</inertial>
 		<visual>
@@ -174,15 +173,14 @@
      </joint>
      <actuator name="j2_motor">
-	    <hardwareInterface>EffortJointInterface</hardwareInterface>
-        <mechanicalReduction>${j2_mechanical_reduction}</mechanicalReduction>
-		<motorTorqueConstant>${j2_motor_torque_constant}</motorTorqueConstant>
-	 </actuator>
+          <mechanicalReduction>${j2_mechanical_reduction}</mechanicalReduction>
+	  <motorTorqueConstant>${j2_motor_torque_constant}</motorTorqueConstant>
+     </actuator>
     </transmission>
     <!-- LINK 3 -->
 	<link name="mico_link_3">
 		<inertial>
-		  <mass value="0.351" />
+		  <mass value="1" />
 		  <origin xyz="-0.07306 0 -0.00466" />
-		  <inertia  ixx="0.0003749308" ixy="0.0"  ixz="-0.0001258961"  iyy="0.0010047174"  iyz="0.0"  izz="0.0009318091" />
+		  <inertia  ixx="0.1" ixy="0.0"  ixz="0.0"  iyy="0.1"  iyz="0.0"  izz="0.1" />
 		</inertial>
 		<visual>
@@ -227,5 +225,4 @@
      </joint>
      <actuator name="j3_motor">
-	    <hardwareInterface>EffortJointInterface</hardwareInterface>
         <mechanicalReduction>${j3_mechanical_reduction}</mechanicalReduction>
 		<motorTorqueConstant>${j3_motor_torque_constant}</motorTorqueConstant>
@@ -235,7 +232,7 @@
 	<link name="mico_link_4">
 		<inertial>
-		  <mass value="0.429" />
-		  <origin xyz="0.06076 0 -0.00014" />
-		  <inertia  ixx="0.0011551458" ixy="-6.3e-010"  ixz="2.519546e-005"  iyy="0.0015754353"  iyz="-7.6e-010"  izz="0.0007798411" />
+		  <mass value="1" />
+		  <origin xyz="0.0 0.0 0.0" />
+		  <inertia  ixx="0.1" ixy="0.0"  ixz="0.0"  iyy="0.1"  iyz="0.0"  izz="0.1" />
 		</inertial>
 		<visual>
@@ -280,5 +277,4 @@
      </joint>
      <actuator name="j4_motor">
-	    <hardwareInterface>EffortJointInterface</hardwareInterface>
         <mechanicalReduction>${j4_mechanical_reduction}</mechanicalReduction>
 		<motorTorqueConstant>${j4_motor_torque_constant}</motorTorqueConstant>
@@ -288,7 +284,7 @@
 	<link name="mico_link_5">
 		<inertial>
-		  <mass value="0.429" />
-		  <origin xyz="0.06076 0 -0.00014" />
-		  <inertia  ixx="0.0011551458" ixy="-6.3e-010"  ixz="2.519546e-005"  iyy="0.0015754353"  iyz="-7.6e-010"  izz="0.0007798411" />
+		  <mass value="1" />
+		  <origin xyz="0.0 0.0 0.0" />
+		  <inertia  ixx="0.1" ixy="0.0"  ixz="0.0"  iyy="0.1"  iyz="0.0"  izz="0.1" />
 		</inertial>
 		<visual>
@@ -333,5 +329,4 @@
      </joint>
      <actuator name="j5_motor">
-	    <hardwareInterface>EffortJointInterface</hardwareInterface>
         <mechanicalReduction>${j5_mechanical_reduction}</mechanicalReduction>
 		<motorTorqueConstant>${j5_motor_torque_constant}</motorTorqueConstant>
@@ -341,7 +336,7 @@
 	<link name="mico_link_hand">
 		<inertial>
-		  <mass value="0.429" />
-		  <origin xyz="0.06076 0 -0.00014" />
-		  <inertia  ixx="0.0011551458" ixy="-6.3e-010"  ixz="2.519546e-005"  iyy="0.0015754353"  iyz="-7.6e-010"  izz="0.0007798411" />
+		  <mass value="1" />
+		  <origin xyz="0.0 0.0 0.0" />
+		  <inertia  ixx="0.1" ixy="0.0"  ixz="0.0"  iyy="0.1"  iyz="0.0"  izz="0.1" />
 		</inertial>
 		<visual>
@@ -386,5 +381,4 @@
      </joint>
      <actuator name="j6_motor">
-	    <hardwareInterface>EffortJointInterface</hardwareInterface>
         <mechanicalReduction>${j6_mechanical_reduction}</mechanicalReduction>
 		<motorTorqueConstant>${j6_motor_torque_constant}</motorTorqueConstant>
@@ -396,5 +390,5 @@
 		  <mass value="0.050" />
 		  <origin xyz="0.03 0.03 0.03" />
-		  <inertia  ixx="0.0011551458" ixy="-6.3e-010"  ixz="2.519546e-005"  iyy="0.0015754353"  iyz="-7.6e-010"  izz="0.0007798411" />
+		  <inertia  ixx="0.0005" ixy="0.0"  ixz="0.0"  iyy="0.0005"  iyz="0.0"  izz="0.0005" />
 		</inertial>
 		<visual>
@@ -439,5 +433,4 @@
      </joint>
      <actuator name="jf1_motor">
-	    <hardwareInterface>EffortJointInterface</hardwareInterface>
         <mechanicalReduction>${jf1_mechanical_reduction}</mechanicalReduction>
 		<motorTorqueConstant>${jf1_motor_torque_constant}</motorTorqueConstant>
@@ -449,5 +442,5 @@
 		  <mass value="0.050" />
 		  <origin xyz="0.03 0.03 0.03" />
-		  <inertia  ixx="0.0011551458" ixy="-6.3e-010"  ixz="2.519546e-005"  iyy="0.0015754353"  iyz="-7.6e-010"  izz="0.0007798411" />
+		  <inertia  ixx="0.0005" ixy="0.0"  ixz="0.0"  iyy="0.0005"  iyz="0.0"  izz="0.0005" />
 		</inertial>
 		<visual>
@@ -492,5 +485,4 @@
      </joint>
      <actuator name="jf2_motor">
-	    <hardwareInterface>EffortJointInterface</hardwareInterface>
         <mechanicalReduction>${jf2_mechanical_reduction}</mechanicalReduction>
 		<motorTorqueConstant>${jf2_motor_torque_constant}</motorTorqueConstant>
