Commit message: modified range of joint 6, -pi/2..3pi/2

File: mico_description/urdf/arms/mico_arm_3fg.urdf.xacro (robot description, xacro)
@@ -29,6 +29,6 @@
 	<xacro:property name="j5_lower_limit" value="-3.13"/>
 	<xacro:property name="j5_upper_limit" value="3.13"/>
-	<xacro:property name="j6_lower_limit" value="-3.13"/>
-	<xacro:property name="j6_upper_limit" value="3.13"/>
+	<xacro:property name="j6_lower_limit" value="-1.52"/>
+	<xacro:property name="j6_upper_limit" value="4.70"/>
 	<xacro:property name="jf1_lower_limit" value="0"/>
 	<xacro:property name="jf1_upper_limit" value="${PI/180*40}"/>

Commit message: updated range of mico 3fg joint 2

File: mico_description/urdf/arms/mico_arm_3fg.urdf.xacro (robot description, xacro)
@@ -22,5 +22,6 @@
 	<xacro:property name="j1_upper_limit" value="3.13"/>
 	<xacro:property name="j2_lower_limit" value="-3.13"/>
-	<xacro:property name="j2_upper_limit" value="0.0"/>
+	<!-- xacro:property name="j2_upper_limit" value="0.0"/ -->
+	<xacro:property name="j2_upper_limit" value="${PI/4}"/>
     <xacro:property name="j3_lower_limit" value="${-5*PI/4}"/>
 	<xacro:property name="j3_upper_limit" value="${PI/4}"/>

Commit message: minor changes in finger inertias to improve dynamic sim in gazebo

File: mico_description/urdf/arms/mico_arm_3fg.urdf.xacro (robot description, xacro)
@@ -2,15 +2,15 @@
 <robot name="mico" xmlns:xacro="http://www.ros.org/wiki/xacro">
  	<xacro:property name="j1_mechanical_reduction" value="1.0"/>
-	<xacro:property name="j1_motor_torque_constant" value="50.0"/>
+	<xacro:property name="j1_motor_torque_constant" value="150.0"/>
 	<xacro:property name="j2_mechanical_reduction" value="1.0"/>
-	<xacro:property name="j2_motor_torque_constant" value="50.0"/>
+	<xacro:property name="j2_motor_torque_constant" value="150.0"/>
 	<xacro:property name="j3_mechanical_reduction" value="1.0"/>
-	<xacro:property name="j3_motor_torque_constant" value="50.0"/>
+	<xacro:property name="j3_motor_torque_constant" value="150.0"/>
 	<xacro:property name="j4_mechanical_reduction" value="1.0"/>
-	<xacro:property name="j4_motor_torque_constant" value="5.0"/>
+	<xacro:property name="j4_motor_torque_constant" value="35.0"/>
 	<xacro:property name="j5_mechanical_reduction" value="1.0"/>
-	<xacro:property name="j5_motor_torque_constant" value="5.0"/>
+	<xacro:property name="j5_motor_torque_constant" value="35.0"/>
 	<xacro:property name="j6_mechanical_reduction" value="1.0"/>
-	<xacro:property name="j6_motor_torque_constant" value="5.0"/>
+	<xacro:property name="j6_motor_torque_constant" value="35.0"/>
 	<xacro:property name="jf1_mechanical_reduction" value="1.0"/>
 	<xacro:property name="jf1_motor_torque_constant" value="5.0"/>
@@ -30,13 +30,8 @@
 	<xacro:property name="j5_lower_limit" value="-3.13"/>
 	<xacro:property name="j5_upper_limit" value="3.13"/>
-	<xacro:property name="j6_lower_limit" value="-1.52"/>
-	<xacro:property name="j6_upper_limit" value="4.70"/>
-	<xacro:property name="jf1_lower_limit" value="0"/>
-	<xacro:property name="jf1_upper_limit" value="${PI/180*40}"/>
-	<xacro:property name="jf2_lower_limit" value="0"/>
-	<xacro:property name="jf2_upper_limit" value="${PI/180*40}"/>
-	<xacro:property name="jf3_lower_limit" value="0"/>
-	<xacro:property name="jf3_upper_limit" value="${PI/180*40}"/>
-	<xacro:property name="joint_effort_limit" value="60.0"/>
+	<xacro:property name="j6_lower_limit" value="-3.13"/>
+	<xacro:property name="j6_upper_limit" value="3.13"/>
+	<!-- xacro:property name="joint_effort_limit" value="60.0"/ -->
+	<xacro:property name="joint_effort_limit" value="80.0"/>
 	<xacro:property name="joint_velocity_limit" value="2.9217"/>
 	<xacro:property name="joint_damping" value="0.7"/>
@@ -69,7 +64,7 @@
 	<link name="mico_link_base">
 		<inertial>
-		  <mass value="0.506" />
-		  <origin xyz="-0.05161 0 -0.003" />
-		  <inertia  ixx="0.0014526484" ixy="0.0"  ixz="-8.792613e-005" iyy="0.0018217854" iyx="0.0"  iyz="0.0" izz="0.0008987159" />
+		  <mass value="1" />
+		  <origin xyz="0.0 0.0 0.0" />
+		  <inertia  ixx="0.1" ixy="0.0"  ixz="0.0" iyy="0.1" iyx="0.0"  iyz="0.0" izz="0.1" />
 		</inertial>
 		<visual>
@@ -99,7 +94,7 @@
     <link name="mico_link_1">
 		<inertial>
-		  <mass value="0.7" />
+		  <mass value="1" />
 		  <origin xyz="0.07155 0.00229 -0.00028" />
-		  <inertia  ixx="0.0018430902" ixy="0.0001075379"  ixz="2.683183e-005"  iyy="0.0023530852"  iyz="4.5192e-007"  izz="0.0016327528" />
+		  <inertia  ixx="0.1" ixy="0.0"  ixz="0.0"  iyy="0.1"  iyz="0.0"  izz="0.1" />
 		</inertial>
 		<visual>
@@ -144,7 +139,6 @@
      </joint>
      <actuator name="j1_motor">
-	    <hardwareInterface>EffortJointInterface</hardwareInterface>
-        <mechanicalReduction>${j1_mechanical_reduction}</mechanicalReduction>
-		<motorTorqueConstant>${j1_motor_torque_constant}</motorTorqueConstant>
+            <mechanicalReduction>${j1_mechanical_reduction}</mechanicalReduction>
+	    <motorTorqueConstant>${j1_motor_torque_constant}</motorTorqueConstant>
 	 </actuator>
     </transmission>
@@ -152,7 +146,7 @@
 	<link name="mico_link_2">
 		<inertial>
-		  <mass value="0.429" />
+		  <mass value="1" />
 		  <origin xyz="0.06076 0 -0.00014" />
-		  <inertia  ixx="0.0011551458" ixy="-6.3e-010"  ixz="2.519546e-005"  iyy="0.0015754353"  iyz="-7.6e-010"  izz="0.0007798411" />
+		  <inertia  ixx="0.1" ixy="0.0"  ixz="0.0"  iyy="0.1"  iyz="0.0"  izz="0.1" />
 		</inertial>
 		<visual>
@@ -197,15 +191,14 @@
      </joint>
      <actuator name="j2_motor">
-	    <hardwareInterface>EffortJointInterface</hardwareInterface>
-        <mechanicalReduction>${j2_mechanical_reduction}</mechanicalReduction>
-		<motorTorqueConstant>${j2_motor_torque_constant}</motorTorqueConstant>
-	 </actuator>
+          <mechanicalReduction>${j2_mechanical_reduction}</mechanicalReduction>
+	  <motorTorqueConstant>${j2_motor_torque_constant}</motorTorqueConstant>
+     </actuator>
     </transmission>
     <!-- LINK 3 -->
 	<link name="mico_link_3">
 		<inertial>
-		  <mass value="0.351" />
+		  <mass value="1" />
 		  <origin xyz="-0.07306 0 -0.00466" />
-		  <inertia  ixx="0.0003749308" ixy="0.0"  ixz="-0.0001258961"  iyy="0.0010047174"  iyz="0.0"  izz="0.0009318091" />
+		  <inertia  ixx="0.1" ixy="0.0"  ixz="0.0"  iyy="0.1"  iyz="0.0"  izz="0.1" />
 		</inertial>
 		<visual>
@@ -250,5 +243,4 @@
      </joint>
      <actuator name="j3_motor">
-	    <hardwareInterface>EffortJointInterface</hardwareInterface>
         <mechanicalReduction>${j3_mechanical_reduction}</mechanicalReduction>
 		<motorTorqueConstant>${j3_motor_torque_constant}</motorTorqueConstant>
@@ -258,7 +250,7 @@
 	<link name="mico_link_4">
 		<inertial>
-		  <mass value="0.429" />
-		  <origin xyz="0.06076 0 -0.00014" />
-		  <inertia  ixx="0.0011551458" ixy="-6.3e-010"  ixz="2.519546e-005"  iyy="0.0015754353"  iyz="-7.6e-010"  izz="0.0007798411" />
+		  <mass value="1" />
+		  <origin xyz="0.0 0.0 0.0" />
+		  <inertia  ixx="0.1" ixy="0.0"  ixz="0.0"  iyy="0.1"  iyz="0.0"  izz="0.1" />
 		</inertial>
 		<visual>
@@ -303,5 +295,4 @@
      </joint>
      <actuator name="j4_motor">
-	    <hardwareInterface>EffortJointInterface</hardwareInterface>
         <mechanicalReduction>${j4_mechanical_reduction}</mechanicalReduction>
 		<motorTorqueConstant>${j4_motor_torque_constant}</motorTorqueConstant>
@@ -311,7 +302,7 @@
 	<link name="mico_link_5">
 		<inertial>
-		  <mass value="0.429" />
-		  <origin xyz="0.06076 0 -0.00014" />
-		  <inertia  ixx="0.0011551458" ixy="-6.3e-010"  ixz="2.519546e-005"  iyy="0.0015754353"  iyz="-7.6e-010"  izz="0.0007798411" />
+		  <mass value="1" />
+		  <origin xyz="0.0 0.0 0.0" />
+		  <inertia  ixx="0.1" ixy="0.0"  ixz="0.0"  iyy="0.1"  iyz="0.0"  izz="0.1" />
 		</inertial>
 		<visual>
@@ -356,5 +347,4 @@
      </joint>
      <actuator name="j5_motor">
-	    <hardwareInterface>EffortJointInterface</hardwareInterface>
         <mechanicalReduction>${j5_mechanical_reduction}</mechanicalReduction>
 		<motorTorqueConstant>${j5_motor_torque_constant}</motorTorqueConstant>
@@ -364,13 +354,13 @@
 	<link name="mico_link_hand">
 		<inertial>
-		  <mass value="0.429" />
-		  <origin xyz="0.06076 0 -0.00014" />
-		  <inertia  ixx="0.0011551458" ixy="-6.3e-010"  ixz="2.519546e-005"  iyy="0.0015754353"  iyz="-7.6e-010"  izz="0.0007798411" />
-		</inertial>
-		<visual>
-		   <origin xyz="0 0 0" rpy="0 0 0" />
-		   <xacro:if value="${hq}">
-		   <geometry>
-			 <mesh filename="package://mico_description/meshes/arms/jaco2_link_hand.dae"/>
+		  <mass value="1" />
+		  <origin xyz="0.0 0.0 0.0" />
+		  <inertia  ixx="0.1" ixy="0.0"  ixz="0.0"  iyy="0.1"  iyz="0.0"  izz="0.1" />
+		</inertial>
+		<visual>
+		   <origin xyz="0 0 0" rpy="0 0 0" />
+		   <xacro:if value="${hq}">
+		   <geometry>
+			 <mesh filename="package://mico_description/meshes/arms/mico_link_hand.dae"/>
 		   </geometry>
 		   </xacro:if>
@@ -387,5 +377,5 @@
 		   <origin xyz="0 0 0" rpy="0 0 0 " />
 		   <geometry>
-		     <mesh filename="package://mico_description/meshes/arms/jaco2_link_hand.dae"/>
+		     <mesh filename="package://mico_description/meshes/arms/mico_link_hand.dae"/>
 		   </geometry>
 		</collision>
@@ -409,5 +399,4 @@
      </joint>
      <actuator name="j6_motor">
-	    <hardwareInterface>EffortJointInterface</hardwareInterface>
         <mechanicalReduction>${j6_mechanical_reduction}</mechanicalReduction>
 		<motorTorqueConstant>${j6_motor_torque_constant}</motorTorqueConstant>
@@ -417,7 +406,7 @@
 	<link name="mico_link_finger_1">
 		<inertial>
-		  <mass value="0.050" />
+		  <mass value="0.10" />
 		  <origin xyz="0.03 0.03 0.03" />
-		  <inertia  ixx="0.0011551458" ixy="-6.3e-010"  ixz="2.519546e-005"  iyy="0.0015754353"  iyz="-7.6e-010"  izz="0.0007798411" />
+		  <inertia  ixx="0.01" ixy="0.0"  ixz="0.0"  iyy="0.01"  iyz="0.0"  izz="0.01" />
 		</inertial>
 		<visual>
@@ -462,5 +451,4 @@
      </joint>
      <actuator name="jf1_motor">
-	    <hardwareInterface>EffortJointInterface</hardwareInterface>
         <mechanicalReduction>${jf1_mechanical_reduction}</mechanicalReduction>
 		<motorTorqueConstant>${jf1_motor_torque_constant}</motorTorqueConstant>
@@ -470,7 +458,7 @@
 	<link name="mico_link_finger_2">
 		<inertial>
-		  <mass value="0.050" />
+		  <mass value="0.10" />
 		  <origin xyz="0.03 0.03 0.03" />
-		  <inertia  ixx="0.0011551458" ixy="-6.3e-010"  ixz="2.519546e-005"  iyy="0.0015754353"  iyz="-7.6e-010"  izz="0.0007798411" />
+		  <inertia  ixx="0.01" ixy="0.0"  ixz="0.0"  iyy="0.01"  iyz="0.0"  izz="0.01" />
 		</inertial>
 		<visual>
@@ -515,5 +503,4 @@
      </joint>
      <actuator name="jf2_motor">
-	    <hardwareInterface>EffortJointInterface</hardwareInterface>
         <mechanicalReduction>${jf2_mechanical_reduction}</mechanicalReduction>
 		<motorTorqueConstant>${jf2_motor_torque_constant}</motorTorqueConstant>
@@ -523,7 +510,7 @@
 	<link name="mico_link_finger_3">
 		<inertial>
-		  <mass value="0.050" />
+		  <mass value="0.1" />
 		  <origin xyz="0.03 0.03 0.03" />
-		  <inertia  ixx="0.0011551458" ixy="-6.3e-010"  ixz="2.519546e-005"  iyy="0.0015754353"  iyz="-7.6e-010"  izz="0.0007798411" />
+		  <inertia  ixx="0.01" ixy="0.0"  ixz="0.0"  iyy="0.01"  iyz="0.0"  izz="0.01" />
 		</inertial>
 		<visual>
@@ -568,5 +555,4 @@
      </joint>
      <actuator name="jf3_motor">
-	    <hardwareInterface>EffortJointInterface</hardwareInterface>
         <mechanicalReduction>${jf3_mechanical_reduction}</mechanicalReduction>
 		<motorTorqueConstant>${jf3_motor_torque_constant}</motorTorqueConstant>

File: mico_description/urdf/arms/mico_arm_rb1.gazebo.xacro (robot description, xacro)
@@ -5,5 +5,4 @@
     <gazebo>
       <plugin name="ros_control" filename="libgazebo_ros_control.so">
-        <!-- robotNamespace>mico</robotNamespace -->
          <robotNamespace>rb1</robotNamespace>
         <robotParam>robot_description</robotParam>
@@ -48,4 +47,8 @@
 		<turnGravityOff>true</turnGravityOff>
 	</gazebo>
+	<gazebo reference="mico_link_finger_3">
+		<material>Gazebo/Grey</material>
+		<turnGravityOff>true</turnGravityOff>
+	</gazebo>
   </xacro:macro>
 </robot>
